Commit message: Add files via upload

File: src/allegro_hand_description/allegro_hand_description_left_A.urdf (robot description, URDF)
Before this commit: robot allegro_hand_left, 22 links, 21 joints
Joints:
- joint joint_0_0: origin xyz=0.0025 -0.034 -0.00945 rpy=0.08726646255 0 0 -> xyz=0.0025 -0.0405 -0.00945 rpy=0.08726646255 0 0
- joint joint_13_0: limit lower=1.57 upper=3.22 effort=15 velocity=7 -> lower=1.4 upper=3.22 effort=15 velocity=7
- joint joint_8_0: origin xyz=0.00 0.034 -0.00945 rpy=-0.08726646255 0 0 -> xyz=0.00 0.0405 -0.00945 rpy=-0.08726646255 0 0

File: src/allegro_hand_description/allegro_hand_description_left_B.urdf (robot description, URDF)
Before this commit: robot allegro_hand_left, 22 links, 21 joints
Joints:
- joint joint_13_0: limit lower=1.57 upper=3.22 effort=15 velocity=7 -> lower=1.4 upper=3.22 effort=15 velocity=7

File: src/allegro_hand_description/allegro_hand_description_right_A.urdf (robot description, URDF)
Before this commit: robot allegro_hand_right, 22 links, 21 joints
Joints:
- joint joint_0_0: origin xyz=0.00 0.0425 -0.00945 rpy=-0.08726646255 0 0 -> xyz=0.00 0.0405 -0.00945 rpy=-0.08726646255 0 0
- joint joint_4_0: origin xyz=0 0.005 -0.0079 rpy=0.0 0 0 -> xyz=0 0.00 -0.0079 rpy=0.0 0 0
- joint joint_8_0: origin xyz=0.0025 -0.036 -0.00945 rpy=0.08726646255 0 0 -> xyz=0.0025 -0.0405 -0.00945 rpy=0.08726646255 0 0

Commit message: Add files via upload

File: src/allegro_hand_description/allegro_hand_description_left_A.urdf (robot description, URDF)
Before this commit: robot allegro_hand_left, 22 links, 21 joints
Joints:
- joint joint_10_0: limit lower=-0.174 upper=1.709 effort=15 velocity=7 -> lower=-0.174 upper=1.9 effort=15 velocity=7
- joint joint_11_0: limit lower=-0.227 upper=1.618 effort=15 velocity=7 -> lower=-0.227 upper=1.9 effort=15 velocity=7
- joint joint_12_0: limit lower=-1.78 upper=0.00 effort=15 velocity=7 -> lower=-1.78 upper=0.5 effort=15 velocity=7
- joint joint_13_0: limit lower=1.4 upper=3.22 effort=15 velocity=7 -> lower=1.0 upper=3.22 effort=15 velocity=7
- joint joint_14_0: limit lower=-1.85 upper=0.05 effort=15 velocity=7 -> lower=-1.85 upper=0.2 effort=15 velocity=7
- joint joint_15_0: limit lower=-1.80 upper=0.09 effort=15 velocity=7 -> lower=-1.80 upper=0.2 effort=15 velocity=7
- joint joint_1_0: limit lower=-0.196 upper=1.61 effort=15 velocity=7 -> lower=-0.196 upper=1.9 effort=15 velocity=7
- joint joint_2_0: limit lower=-0.174 upper=1.709 effort=15 velocity=7 -> lower=-0.174 upper=1.9 effort=15 velocity=7
- joint joint_3_0: limit lower=-0.227 upper=1.618 effort=15 velocity=7 -> lower=-0.227 upper=1.9 effort=15 velocity=7
- joint joint_5_0: limit lower=-0.196 upper=1.61 effort=15 velocity=7 -> lower=-0.196 upper=1.9 effort=15 velocity=7
- joint joint_6_0: limit lower=-0.174 upper=1.709 effort=15 velocity=7 -> lower=-0.174 upper=1.9 effort=15 velocity=7
- joint joint_7_0: limit lower=-0.227 upper=1.618 effort=15 velocity=7 -> lower=-0.227 upper=1.9 effort=15 velocity=7
- joint joint_9_0: limit lower=-0.196 upper=1.61 effort=15 velocity=7 -> lower=-0.196 upper=1.9 effort=15 velocity=7

File: src/allegro_hand_description/allegro_hand_description_left_B.urdf (robot description, URDF)
Before this commit: robot allegro_hand_left, 22 links, 21 joints
Joints:
- joint joint_12_0: limit lower=-1.78 upper=0.00 effort=15 velocity=7 -> lower=-1.78 upper=0.5 effort=15 velocity=7
- joint joint_13_0: limit lower=1.4 upper=3.22 effort=15 velocity=7 -> lower=1.0 upper=3.22 effort=15 velocity=7
- joint joint_14_0: limit lower=-1.85 upper=0.05 effort=15 velocity=7 -> lower=-1.85 upper=0.2 effort=15 velocity=7
- joint joint_15_0: limit lower=-1.80 upper=0.09 effort=15 velocity=7 -> lower=-1.80 upper=0.2 effort=15 velocity=7

Commit message: Add files via upload

File: src/allegro_hand_description/allegro_hand_description_left_A.urdf (robot description, URDF)
Before this commit: robot allegro_hand_left, 22 links, 21 joints
Links:
- link link_0_0: mass 0.0119 -> 0.0176
- link link_10_0: mass 0.0355 -> 0.0366
- link link_11_0: mass 0.0096 -> 0.00569
- link link_11_0_tip: mass 0.0168 -> 0.00
- link link_1_0: mass 0.065 -> 0.066
- link link_2_0: mass 0.0355 -> 0.0366
- link link_3_0: mass 0.0096 -> 0.00569
- link link_3_0_tip: mass 0.0168 -> 0.00
- link link_4_0: mass 0.0119 -> 0.0176
- link link_5_0: mass 0.065 -> 0.066
- link link_6_0: mass 0.0355 -> 0.0366
- link link_7_0: mass 0.0096 -> 0.00569
- link link_7_0_tip: mass 0.0168 -> 0.00
- link link_8_0: mass 0.0119 -> 0.0176
- link link_9_0: mass 0.065 -> 0.066

File: src/allegro_hand_description/allegro_hand_description_right_A.urdf (robot description, URDF)
Before this commit: robot allegro_hand_right, 22 links, 21 joints
Links:
- link link_0_0: mass 0.0119 -> 0.0176
- link link_10_0: mass 0.0355 -> 0.0366
- link link_11_0: mass 0.0096 -> 0.00569
- link link_11_0_tip: mass 0.0168 -> 0.00
- link link_15_0: mass 0.0334 -> 0.0338
- link link_15_0_tip: mass 0.0014 -> 0.00
- link link_1_0: mass 0.065 -> 0.066
- link link_2_0: mass 0.0355 -> 0.0366
- link link_3_0: mass 0.0096 -> 0.00569
- link link_3_0_tip: mass 0.0168 -> 0.00
- link link_4_0: mass 0.0119 -> 0.0176
- link link_5_0: mass 0.065 -> 0.066
- link link_6_0: mass 0.0355 -> 0.0366
- link link_7_0: mass 0.0096 -> 0.00569
- link link_7_0_tip: mass 0.0168 -> 0.00
- link link_8_0: mass 0.0119 -> 0.0176
- link link_9_0: mass 0.065 -> 0.066
